Commit message: Zed fully resolved

File: zed_wrapper/urdf/zed_descr.urdf.xacro (robot description, xacro)
@@ -16,6 +16,6 @@
 -->
 <robot name="stereolabs_camera" xmlns:xacro="http://ros.org/wiki/xacro">
-  <xacro:arg name="camera_name"   default="zed" />
-  <xacro:arg name="camera_model"  default="zed" />
+  <xacro:arg name="camera_name"   default="zed2i" />
+  <xacro:arg name="camera_model"  default="zed2i" />
   <xacro:arg name="base_frame"    default="base_link" />
   <xacro:arg name="cam_pos_x"     default="0.0" />

File: zed_wrapper/urdf/zed_macro.urdf.xacro (robot description, xacro)
@@ -127,4 +127,11 @@
       <child link="${name}_right_camera_optical_frame"/>
     </joint>
+  <!-- IMU -->
+  <!--   rotation:
+    x: -0.00183512
+    y: 0.000211432
+    z: -0.00651105
+    w: 0.999977
+ -->
   <xacro:if value="${model == 'zed2i'}">
     <link name="zed2i_imu_link" />
@@ -132,5 +139,5 @@
       <parent link="zed2i_left_camera_frame"/>
       <child link="zed2i_imu_link"/>
-      <origin xyz="-0.002000 -0.023061 0.000217" rpy="-0.0036659 0.0004207 -0.0130222" />
+      <origin xyz="-0.002000 -0.023061 0.000217" rpy="-0.00367291 0.00039895 -0.013022948" />
     </joint>
   </xacro:if>
